File: QuadLevelShifter.kicad_pcb (KiCad board)
At the start: 4 copper layers, 52 x 35.9 mm, 52 parts, among them P1 EDGE_CONN_02X09, Q1 BSS138, Q2 BSS138, Q3 BSS138, Q4 BSS138, U1 2EDN7524, U2 MAX395CWG+, U3 2EDN7524, U4 2EDN7524, U5 2EDN7524

Commit message: First attempt at PCB
Parts:
- added REF**: CC-BY-SA Logo, CC-BY-SA_Logo, F.Cu at (0.00, 0.00)
- added REF**: CC-BY-SA Logo, quad_level_shifter:CC-BY-SA_Logo, B.Cu at (104.4, 95.0)
- added REF***: OSHW-Logo_5.7x6mm_SilkScreen, Symbols:OSHW-Logo_5.7x6mm_SilkScreen, B.Cu at (116.3, 90.5)
- moved D14 1.30 mm to (118.9, 92.5)
- moved D16 1.30 mm to (118.9, 105.2)
- moved D10 1.27 mm to (117.6, 92.5)
- moved D12 1.27 mm to (117.6, 105.2)
- moved D8 1.27 mm to (73.5, 85.1)
- moved D6 1.24 mm to (73.5, 97.9)
- moved D2 1.23 mm to (74.7, 97.9)
- moved D4 1.20 mm to (74.7, 85.1)
Routing:
- net GND: track 6.45 -> 46.2 mm, vias 1 -> 16
- net VDD: track 3.21 -> 41.4 mm, vias 1 -> 14
- net +12V: track 3.00 -> 39.1 mm, vias 1 -> 15
- net /IO2_HV_DR: track 0.00 -> 9.10 mm
- net /IO0_HV_DR: track 0.00 -> 8.95 mm
- net /IO0_LV_DR: track 0.00 -> 8.73 mm
- net /IO2_LV_DR: track 0.00 -> 8.62 mm
- net /IO3_HV_DR: track 0.00 -> 4.76 mm
- net /IO1_HV_DR: track 0.00 -> 4.76 mm
- net /IO3_LV_DR: track 0.00 -> 4.64 mm
- net /IO1_LV_DR: track 0.00 -> 4.64 mm
- net /CS: track 38.3 -> 35.8 mm
- net DOUT: track 29.5 -> 30.5 mm
- net /IO3_LV_SW: track 49.9 -> 49.0 mm
- net /IO2_HV_SW: track 43.9 -> 44.6 mm
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Other:
- board text added: "+12V"
- board text added: "-CS"
- board text added: "-RST"
- board text added: "2EDN7524"
- board text added: "DIN"
- board text added: "DOUT"
- board text added: "GND"
- board text added: "IO0_HV"
- board text added: "IO0_LV"
- board text added: "IO1_HV"
- board text added: "IO1_LV"
- board text added: "IO2_HV"
- board text added: "IO2_LV"
- board text added: "IO3_HV"
- board text added: "IO3_LV"
- board text added: "MAX395"
- board text added: "N/C"
- board text added: "QUAD LV/HV LEVEL SHIFTER REV A 2016 DEC 4"
- board text added: "SCLK"
- board text added: "VDD"
- board text added: "github.com/RobertBaruch/QuadLevelShifter"

Commit message: Completed revision A
Parts:
- removed the REF** at (0.00, 0.00)
- removed the REF*** at (116.3, 90.5)
- added C11: 10u, quad_level_shifter:c_elec_6.3x5.3, F.Cu at (75.6, 112.2)
- added C12: 10u, quad_level_shifter:c_elec_6.3x5.3, F.Cu at (116.2, 112.0)
- added REF***: OSHW-Symbol_6.7x6mm_SilkScreen, Symbols:OSHW-Symbol_6.7x6mm_SilkScreen, B.Cu at (117.4, 89.8)
Routing:
- net GND: track 46.2 -> 57.5 mm, vias 16 -> 22
- net VDD: track 41.4 -> 48.6 mm, vias 14 -> 17
- net +12V: track 39.1 -> 45.0 mm, vias 15 -> 18
Other:
- board text added: "QUAD LV/HV LEVEL SHIFTER REV A 2016 DEC 8"
- board text added: "SPBC"
- board text removed: "QUAD LV/HV LEVEL SHIFTER REV A 2016 DEC 4"
