File: QuadLevelShifter.sch (KiCad schematic (older format))
At the start: 52 parts, among them P1 EDGE_CONN_02X09, Q1 BSS138, Q2 BSS138, Q3 BSS138, Q4 BSS138, U1 2EDN7524, U2 MAX395CWG+, U3 2EDN7524, U4 2EDN7524, U5 2EDN7524

Commit message: Completed revision A
Parts:
- added C11, C12: 10u, quad_level_shifter:c_elec_6.3x5.3, symbol 10u
Connections:
- net +12V: now also C11.1
- net GNDREF: now also C11.2, C12.2
- net VDD: now also C12.1
Other:
- note added: "This work is licensed under the Creative Commons Attribution-\nShareAlike 4.0 International License. To view a copy of this license,\nvisit http://creativecommons.org/licenses/by-sa/4.0/ or send a letter\nto Creative Commons, PO Box 1866, Mountain View, CA 94042, USA.\n\nAttribution: Robert Baruch (robert.c.baruch@gmail.com)"
